Commit message: added euslisp scripts for plugin utility

File: hrpsys_gazebo_tutorials/environment_models/simple-box/model.urdf (robot description, URDF)
Before this commit: robot simple-box-robot, 1 links, 0 joints
Links:
- link nil_link: mass 20 -> 2

Commit message: changed box size for simple-box-for-holding

File: hrpsys_gazebo_tutorials/environment_models/simple-box/model.urdf (robot description, URDF)
Before this commit: robot simple-box-robot, 1 links, 0 joints
Links:
- link nil_link: geometry collision box size=0.25 0.5 0.35; visual box size=0.25 0.5 0.35
