Commit message: update hand model

File: hrpsys_gazebo_atlas/models/sandia_hand_left.urdf (robot description, URDF)
Before this commit: robot sandia_hand_left, 34 links, 33 joints
Joints:
- joint left_sandia_hand_joint: origin xyz=0  0.1 0 rpy= 1.57079 0  1.57079 -> xyz=0.00179  0.13516 0.01176 rpy=0 0  1.57079

File: hrpsys_gazebo_atlas/models/sandia_hand_right.urdf (robot description, URDF)
Before this commit: robot sandia_hand_right, 34 links, 33 joints
Joints:
- joint right_sandia_hand_joint: origin xyz=0 -0.1 0 rpy=-1.57079 0 -1.57079 -> xyz=-0.00179 -0.13516 0.01176 rpy=0 0 -1.57079
