Commit message: fix collision mesh of hook hand model

File: hrpsys_gazebo_atlas/models/hook_hand.urdf.xacro (robot description, xacro)
@@ -14,5 +14,5 @@
 	<origin xyz="0 0 0" rpy = "0 1.57 0" />
 	<geometry>
-	  <mesh filename="package://hrpsys_gazebo_atlas/models/meshes/hook_collision.dae" scale= ".001 .001 .001"/>
+	  <mesh filename="package://hrpsys_gazebo_atlas/models/hook_collision.dae" scale= "1.0 1.0 1.0"/>
 	</geometry>
       </collision>
