Commit message: add kinect by sed command instead of xacro: hector_sensors_description is unneeded.

File: hrpsys_gazebo_tutorials/robot_models/HRP2JSKNT/HRP2JSKNT.urdf.xacro (robot description, xacro)
@@ -4,8 +4,3 @@
   <xacro:include filename="$(find hrpsys_gazebo_tutorials)/robot_models/HRP3HAND_R/HRP3HAND_R.urdf" />
   <include filename="$(find hector_sensors_description)/urdf/asus_camera.urdf.xacro" />
-  <xacro:asus_camera name="xtion" parent="HEAD_LINK1">
-    <origin xyz="0.1120 0.0 0.1255" rpy="0 0 0"/>
-    <!-- origin is calculated from -->
-    <!-- (send (send (send *hrp2jsknt* :head_link1_lk) :worldcoords) :transformation (midcoords 0.5 (send *hrp2jsknt* :camera_l) (send *hrp2jsknt* :camera_r))) -->
-  </xacro:asus_camera>
 </robot>

Commit message: added kinect and hand end effector by xacro instead of sed

File: hrpsys_gazebo_tutorials/robot_models/HRP2JSKNT/HRP2JSKNT.urdf.xacro (robot description, xacro)
@@ -3,3 +3,97 @@
   <xacro:include filename="$(find hrpsys_gazebo_tutorials)/robot_models/HRP3HAND_L/HRP3HAND_L.urdf" />
   <xacro:include filename="$(find hrpsys_gazebo_tutorials)/robot_models/HRP3HAND_R/HRP3HAND_R.urdf" />
+  <!-- add Kinect plugin, link and joint without visual and collision -->
+  <joint name="xtion_joint" type="fixed">
+    <origin rpy="0 0 0" xyz="0.1120 0.0 0.1255"/>
+    <parent link="HEAD_LINK1"/>
+    <child link="xtion_link"/>
+  </joint>
+  <link name="xtion_link">
+    <inertial>
+      <mass value="0.200"/>
+      <origin rpy="0 0 0" xyz="0 0 0"/>
+      <inertia ixx="5.8083e-4" ixy="0" ixz="0" iyy="3.0833e-5" iyz="0" izz="5.9083e-4"/>
+    </inertial>
+  </link>
+  <joint name="xtion_depth_joint" type="fixed">
+    <origin rpy="0 0 0" xyz="0.0 0.049 0.0"/>
+    <parent link="xtion_link"/>
+    <child link="xtion_depth_frame"/>
+  </joint>
+  <link name="xtion_depth_frame"/>
+  <joint name="xtion_depth_optical_joint" type="fixed">
+    <origin rpy="-1.57079632679 0.0 -1.57079632679" xyz="0 0 0"/>
+    <parent link="xtion_depth_frame"/>
+    <child link="xtion_depth_optical_frame"/>
+  </joint>
+  <link name="xtion_depth_optical_frame"/>
+  <joint name="xtion_rgb_joint" type="fixed">
+    <origin rpy="0 0 0" xyz="0.0 0.022 0.0"/>
+    <parent link="xtion_link"/>
+    <child link="xtion_rgb_frame"/>
+  </joint>
+  <link name="xtion_rgb_frame"/>
+  <joint name="xtion_rgb_optical_joint" type="fixed">
+    <origin rpy="-1.57079632679 0.0 -1.57079632679" xyz="0 0 0"/>
+    <parent link="xtion_rgb_frame"/>
+    <child link="xtion_rgb_optical_frame"/>
+  </joint>
+  <link name="xtion_rgb_optical_frame"/>
+  <gazebo reference="xtion_depth_frame">
+    <sensor name="xtion" type="depth">
+      <update_rate>20</update_rate>
+      <camera>
+        <horizontal_fov>1.09606677025</horizontal_fov>
+        <image>
+          <format>R8G8B8</format>
+          <width>640</width>
+          <height>480</height>
+        </image>
+        <clip>
+          <near>0.5</near>
+          <far>9</far>
+        </clip>
+      </camera>
+      <plugin filename="libgazebo_ros_openni_kinect.so" name="xtion_camera_controller">
+        <alwaysOn>true</alwaysOn>
+        <updateRate>20</updateRate>
+        <imageTopicName>xtion/rgb/image_raw</imageTopicName>
+        <cameraInfoTopicName>xtion/rgb/camera_info</cameraInfoTopicName>
+        <depthImageTopicName>xtion/depth/image_raw</depthImageTopicName>
+        <depthImageCameraInfoTopicName>xtion/depth/camera_info</depthImageCameraInfoTopicName>
+        <pointCloudTopicName>xtion/depth/points</pointCloudTopicName>
+        <frameName>xtion_depth_optical_frame</frameName>
+        <distortion_k1>0.0</distortion_k1>
+        <distortion_k2>0.0</distortion_k2>
+        <distortion_k3>0.0</distortion_k3>
+        <distortion_t1>0.0</distortion_t1>
+        <distortion_t2>0.0</distortion_t2>
+      </plugin>
+    </sensor>
+  </gazebo>
+  <!-- added end-effector virtual joints and links -->
+  <link name="RARM_EEF_PARENT" />
+  <link name="RARM_EEF_CHILD" />
+  <joint name="rarm_eef_1" type="fixed">
+    <origin rpy="0 1.5708 0" xyz="-0.0042 0.0392 -0.1245"/>
+    <parent link="RARM_LINK6"/>
+    <child link="RARM_EEF_PARENT"/>
+  </joint>
+  <joint name="rarm_eef_2" type="fixed">
+    <origin rpy="0 0 0" xyz="0 0 0"/>
+    <parent link="RARM_EEF_PARENT"/>
+    <child link="RARM_EEF_CHILD"/>
+  </joint>
+  <link name="LARM_EEF_PARENT" />
+  <link name="LARM_EEF_CHILD" />
+  <joint name="larm_eef_1" type="fixed">
+    <origin rpy="0 1.5708 0" xyz="-0.0042 -0.0392 -0.1245"/>
+    <parent link="LARM_LINK6"/>
+    <child link="LARM_EEF_PARENT"/>
+  </joint>
+  <joint name="larm_eef_2" type="fixed">
+    <origin rpy="0 0 0" xyz="0 0 0"/>
+    <parent link="LARM_EEF_PARENT"/>
+    <child link="LARM_EEF_CHILD"/>
+  </joint>
 </robot>

File: hrpsys_gazebo_tutorials/robot_models/HRP2JSKNTS/HRP2JSKNTS.urdf.xacro (robot description, xacro)
@@ -3,3 +3,97 @@
   <xacro:include filename="$(find hrpsys_gazebo_tutorials)/robot_models/HRP3HAND_L/HRP3HAND_L.urdf" />
   <xacro:include filename="$(find hrpsys_gazebo_tutorials)/robot_models/HRP3HAND_R/HRP3HAND_R.urdf" />
+  <!-- add Kinect plugin, link and joint without visual and collision -->
+  <joint name="xtion_joint" type="fixed">
+    <origin rpy="0 0 0" xyz="0.1120 0.0 0.1255"/>
+    <parent link="HEAD_LINK1"/>
+    <child link="xtion_link"/>
+  </joint>
+  <link name="xtion_link">
+    <inertial>
+      <mass value="0.200"/>
+      <origin rpy="0 0 0" xyz="0 0 0"/>
+      <inertia ixx="5.8083e-4" ixy="0" ixz="0" iyy="3.0833e-5" iyz="0" izz="5.9083e-4"/>
+    </inertial>
+  </link>
+  <joint name="xtion_depth_joint" type="fixed">
+    <origin rpy="0 0 0" xyz="0.0 0.049 0.0"/>
+    <parent link="xtion_link"/>
+    <child link="xtion_depth_frame"/>
+  </joint>
+  <link name="xtion_depth_frame"/>
+  <joint name="xtion_depth_optical_joint" type="fixed">
+    <origin rpy="-1.57079632679 0.0 -1.57079632679" xyz="0 0 0"/>
+    <parent link="xtion_depth_frame"/>
+    <child link="xtion_depth_optical_frame"/>
+  </joint>
+  <link name="xtion_depth_optical_frame"/>
+  <joint name="xtion_rgb_joint" type="fixed">
+    <origin rpy="0 0 0" xyz="0.0 0.022 0.0"/>
+    <parent link="xtion_link"/>
+    <child link="xtion_rgb_frame"/>
+  </joint>
+  <link name="xtion_rgb_frame"/>
+  <joint name="xtion_rgb_optical_joint" type="fixed">
+    <origin rpy="-1.57079632679 0.0 -1.57079632679" xyz="0 0 0"/>
+    <parent link="xtion_rgb_frame"/>
+    <child link="xtion_rgb_optical_frame"/>
+  </joint>
+  <link name="xtion_rgb_optical_frame"/>
+  <gazebo reference="xtion_depth_frame">
+    <sensor name="xtion" type="depth">
+      <update_rate>20</update_rate>
+      <camera>
+        <horizontal_fov>1.09606677025</horizontal_fov>
+        <image>
+          <format>R8G8B8</format>
+          <width>640</width>
+          <height>480</height>
+        </image>
+        <clip>
+          <near>0.5</near>
+          <far>9</far>
+        </clip>
+      </camera>
+      <plugin filename="libgazebo_ros_openni_kinect.so" name="xtion_camera_controller">
+        <alwaysOn>true</alwaysOn>
+        <updateRate>20</updateRate>
+        <imageTopicName>xtion/rgb/image_raw</imageTopicName>
+        <cameraInfoTopicName>xtion/rgb/camera_info</cameraInfoTopicName>
+        <depthImageTopicName>xtion/depth/image_raw</depthImageTopicName>
+        <depthImageCameraInfoTopicName>xtion/depth/camera_info</depthImageCameraInfoTopicName>
+        <pointCloudTopicName>xtion/depth/points</pointCloudTopicName>
+        <frameName>xtion_depth_optical_frame</frameName>
+        <distortion_k1>0.0</distortion_k1>
+        <distortion_k2>0.0</distortion_k2>
+        <distortion_k3>0.0</distortion_k3>
+        <distortion_t1>0.0</distortion_t1>
+        <distortion_t2>0.0</distortion_t2>
+      </plugin>
+    </sensor>
+  </gazebo>
+  <!-- added end-effector virtual joints and links -->
+  <link name="RARM_EEF_PARENT" />
+  <link name="RARM_EEF_CHILD" />
+  <joint name="rarm_eef_1" type="fixed">
+    <origin rpy="0 1.5708 0" xyz="-0.0042 0.0392 -0.1245"/>
+    <parent link="RARM_LINK6"/>
+    <child link="RARM_EEF_PARENT"/>
+  </joint>
+  <joint name="rarm_eef_2" type="fixed">
+    <origin rpy="0 0 0" xyz="0 0 0"/>
+    <parent link="RARM_EEF_PARENT"/>
+    <child link="RARM_EEF_CHILD"/>
+  </joint>
+  <link name="LARM_EEF_PARENT" />
+  <link name="LARM_EEF_CHILD" />
+  <joint name="larm_eef_1" type="fixed">
+    <origin rpy="0 1.5708 0" xyz="-0.0042 -0.0392 -0.1245"/>
+    <parent link="LARM_LINK6"/>
+    <child link="LARM_EEF_PARENT"/>
+  </joint>
+  <joint name="larm_eef_2" type="fixed">
+    <origin rpy="0 0 0" xyz="0 0 0"/>
+    <parent link="LARM_EEF_PARENT"/>
+    <child link="LARM_EEF_CHILD"/>
+  </joint>
 </robot>
